Commit message: fix: Use cylinder instead of original mesh for wheel collision geometry

File: resources/robots/wheel_legged_universal/urdf/universal.urdf (robot description, URDF)
Before this commit: robot universal, 7 links, 6 joints
Links:
- link left_wheel: geometry collision cylinder length=0.025 radius=0.06; visual mesh filename=../meshes/left_wheel.STL
- link right_wheel: geometry collision cylinder length=0.025 radius=0.06; visual mesh filename=../meshes/right_wheel.STL
Joints:
- joint left_knee: limit lower=0 upper=1.1414 effort=40 velocity=1000 -> lower=0 upper=1.1414 effort=60 velocity=1000
- joint right_knee: limit lower=0 upper=1.1414 effort=40 velocity=1000 -> lower=0 upper=1.1414 effort=60 velocity=1000

Commit message: para: limit wheel joint effort to real max torque

File: resources/robots/wheel_legged_universal/urdf/universal.urdf (robot description, URDF)
Before this commit: robot universal, 7 links, 6 joints
Joints:
- joint left_wheel_axis: limit effort=5 velocity=1000 -> effort=3.8 velocity=1000
- joint right_wheel_axis: limit effort=5 velocity=1000 -> effort=3.8 velocity=1000
